Commit message: fixed (changed px4 also) - ros2_control + px4 + gz

File: src/darm/urdf/x500_base/control.xacro (robot description, xacro)
@@ -2,10 +2,15 @@
 <robot xmlns:xacro="http://ros.org/wiki/xacro">
   <!-- Macro to declare ros2_control system -->
-    <xacro:macro name="ros2_control_block" params="joint_name">
-        <!-- Loop through all provided joints -->
-        <joint name="${joint_name}" >
-            <command_interface name="position"/>
-            <state_interface name="position"/>
-        </joint>
+    <xacro:macro name="arm_joint_control" params="joint_name link_name">
+        <transmission name="${joint_name}_transmission">
+            <type>transmission_interface/SimpleTransmission</type>
+            <joint name="${joint_name}">
+            <hardwareInterface>position</hardwareInterface>
+            </joint>
+            <actuator name="${link_name}">
+            <hardwareInterface>position</hardwareInterface>
+            <mechanicalReduction>1</mechanicalReduction>
+            </actuator>
+        </transmission>
     </xacro:macro>
 </robot>

File: src/darm/urdf/x500_base/model.xacro (robot description, xacro)
@@ -4,5 +4,5 @@
   <xacro:include filename="materials.xacro"/>
   <xacro:include filename="control.xacro"/>
-  <xacro:property name="mesh_prefix" value="package://darm/urdf"/>
+  <xacro:property name="mesh_prefix" value="file://$(find darm)/models"/>
   <link name="base_link">
     <inertial>
@@ -244,4 +244,5 @@
       <limit lower="-3.14" upper="3.14" effort="1" velocity="1"/>
   </joint>
+  <xacro:arm_joint_control joint_name="joint1" link_name="link1"/>
   <link name="link_sphere">
       <visual>
@@ -267,4 +268,5 @@
       <limit lower="-3.14" upper="3.14" effort="1" velocity="1"/>
   </joint>
+  <xacro:arm_joint_control joint_name="joint2" link_name="link_sphere"/>
   <link name="link2">
       <visual>

File: src/darm/urdf/x500_base/robot.urdf.xacro (robot description, xacro)
@@ -4,8 +4,8 @@
   <xacro:include filename="macros.xacro"/>
   <xacro:include filename="control.xacro"/>
-  <gazebo>
+  <!-- <gazebo>
     <plugin filename="gz_ros2_control-system" name="gz_ros2_control::GazeboSimROS2ControlPlugin">
       <parameters>package://darm/config/arm_control.yaml</parameters>
     </plugin>
-  </gazebo>
+  </gazebo> -->
 </robot>
