Commit message: setup effort controller also

File: src/darm/urdf/x500_base/model.xacro (robot description, xacro)
@@ -295,4 +295,18 @@
         <plugin>gz_ros2_control/GazeboSimSystem</plugin>
     </hardware>
+    <!-- chose this for effort controller -->
+    <!-- <joint name = "joint1">
+      <command_interface name = "effort"/>
+      <state_interface name = "position"/>
+      <state_interface name = "velocity"/>
+      <state_interface name = "effort"/>
+    </joint>
+    <joint name = "joint2">
+      <command_interface name = "effort"/>
+      <state_interface name = "position"/>
+      <state_interface name = "velocity"/>
+      <state_interface name = "effort"/>
+    </joint> -->
+    <!-- this for position controller -->
     <joint name = "joint1">
       <command_interface name = "position"/>
